Commit message: 使用 slam_tool

File: urdf/robot.urdf (robot description, URDF)
Before this commit: robot omni_robot, 6 links, 5 joints
Links:
- link base_link: geometry collision box size=0.262 0.270 0.050; visual box size=0.262 0.270 0.050

Commit message: refactor: 切换到Cartographer实时建图方案
- 移除 slam_toolbox 配置和定位模式
- 移除 ICP 重定位脚本
- 更新 Cartographer 配置为实时建图模式
- 简化 launch 文件，移除重复节点
- 禁用里程计的 SLAM 校正（Cartographer 内部融合）
- 删除预建图文件（不再需要）

File: urdf/robot.urdf (robot description, URDF)
Before this commit: robot omni_robot, 6 links, 5 joints
Links:
- link base_link: geometry collision box size=0.382 0.340 0.050; visual box size=0.342 0.300 0.050
